File: electronics/PIDriverElectronics.kicad_sch (KiCad schematic)
At the start: 0 parts

Commit message: begin electronics kicad project and add .gitignore for kicad files
Other:
- company: (none) -> BreadLeaf Projects
- title: (none) -> PIDriver
